Commit message: Added simple shape
added link and joint of simple shape to file

File: omtp_factory.xacro (robot description, xacro)
@@ -11,4 +11,25 @@
     <origin xyz="0.5 1.8 0.0" rpy="0 0 0"/>
   </xacro:robot_pedestal_urdf>
+  <!-- simple shape -->
+  <xacro:property name="h" value="1.8" />
+  <xacro:property name="l" value="0.5" />
+  <xacro:property name="d" value="0.2" />
+  <material name="green">
+    <color rgba="0 1 0 1"/>
+  </material>
+  <link name="SimpleShape" >
+    <visual>
+    <geometry>
+     <box size="${l} ${d} ${h}"/>
+    </geometry>
+    <origin rpy="0 0 0" xyz="${l/2} ${d/2} 0"/>
+    <material name="green"/>
+    <collision>
+        <geometry>
+            <box size="${l} ${d} ${h}"/>
+        </geometry>
+    </collision>
+    </visual>
+  </link>
   <!-- Robot1 -->
   <xacro:include filename="$(find ur_description)/urdf/ur10.urdf.xacro"/>
@@ -24,4 +45,10 @@
     <parent link="world" />
     <child link="world_interface" />
+  </joint>
+ <!-- SimpleShape to world. -->
+  <joint name="SimpleShape_to_world_interface" type="fixed">
+    <parent link="world_interface" />
+    <child link="SimpleShape" />
+    <origin xyz="-3 -0.5 0.0" rpy="0.0 0.0 0.0"/>
   </joint>
   <!-- robot1-pedestal to world. -->

Commit message: Added UR5 and ABB robot
Added a second UR5 and a ABB robot to the environment

File: omtp_factory.xacro (robot description, xacro)
@@ -10,4 +10,8 @@
   <xacro:robot_pedestal_urdf pedestal_prefix="robot1_" pedestal_parent="world_interface" pedestal_height="0.95">
     <origin xyz="0.5 1.8 0.0" rpy="0 0 0"/>
+  </xacro:robot_pedestal_urdf>
+  <!-- Robot2 Pedestal -->
+  <xacro:robot_pedestal_urdf pedestal_prefix="robot2_" pedestal_parent="world_interface" pedestal_height="0.95">
+    <origin xyz="1.5 1.8 1.0" rpy="0 0 0"/>
   </xacro:robot_pedestal_urdf>
   <!-- simple shape -->
@@ -41,4 +45,7 @@
   <xacro:include filename="$(find omtp_support)/urdf/bin/bin.urdf.xacro"/>
   <xacro:bin_urdf prefix="bin_1_"/>
+  <!-- ABB robot -->
+  <xacro:include filename="$(find abb_irb6600_support)/urdf/irb6640_macro.xacro"/>
+  <xacro:abb_irb6640 prefix="ABB_"/>
   <!-- Joints -->
   <joint name="world_interface_to_world" type="fixed">
@@ -57,4 +64,16 @@
     <child link="robot1_pedestal_link" />
     <origin xyz="0.5 1.8 0.0" rpy="0.0 0.0 0.0"/>
+  </joint>
+ <!-- robot2-pedestal to world. -->
+  <joint name="robot2_pedestal_to_world_interface" type="fixed">
+    <parent link="world_interface" />
+    <child link="robot2_pedestal_link" />
+    <origin xyz="2.5 1.8 0.0" rpy="0.0 0.0 0.0"/>
+  </joint>
+  <!-- robot2 to pedestal. -->
+  <joint name="robot2_to_pedestal" type="fixed">
+  <origin xyz="0 0 0.95" rpy="0 0 0" />
+  <parent link="robot2_pedestal_link" />
+  <child link="robot2_base_link" />
   </joint>
   <!-- robot1 to pedestal. -->
@@ -75,3 +94,9 @@
     <origin xyz="-7.5 -0.3 0.0" rpy="0 0 0" />
   </joint>
+  <!-- ABB to world. -->
+  <joint name="ABB_to_world_interface" type="fixed">
+    <parent link="world_interface" />
+    <child link="ABB_base_link" />
+    <origin xyz="0.24 -5 0.0" rpy="0.0 0.0 0.0"/>
+  </joint>
 </robot>
